File: pcb/main_board/main_board.kicad_pcb (KiCad board)
At the start: 2 copper layers, 100.3 x 100.3 mm, 36 parts, among them J1 Sensors_Conn, J2 Power_Conn, J3 I2C_Conn, J4 Garage_Conn, J5 Debug_Sensors_Conn, J6 Debug_I2C_Conn, U1 ESP-01, U2 HC_05, U3 AT24CS64-SSHM, U4 AMS1117-3.3, U5 Black_Pill

Commit message: Main board PCB updated
Parts:
- J3: footprint Connector_IDC:IDC-Header_2x04_P2.54mm_Vertical -> Connector_IDC:IDC-Header_2x03_P2.54mm_Vertical
- moved R4 7.88 mm to (122.4, 106.9), turned to 0 degrees
- moved J2 7.15 mm to (123.7, 71.6)
- moved R14 3.56 mm to (165.6, 96.8)
- moved R16 3.56 mm to (165.6, 94.0)
- moved REF** 3.05 mm to (192.3, 72.1)
- moved REF** 3.05 mm to (111.0, 72.1)
- moved C1 0.51 mm to (107.2, 89.2)
Connections:
- U2 pad 1: BT_KEY -> Net-(U2-Pad1)
- U2 pad 2: 5V -> BT_RX_STM_TX
- U2 pad 3: GND -> BT_TX_STM_RX
- U2 pad 4: BT_TX_STM_RX -> GND
- U2 pad 5: BT_RX_STM_TX -> 5V
- U2 pad 6: Net-(U2-Pad6) -> BT_KEY
Routing:
- net BT_RX_STM_TX: track 27.1 -> 45.0 mm
- net BT_KEY: track 36.7 -> 25.5 mm
- net 5V: track 191.5 -> 196.1 mm
- net Net-(R14-Pad2): track 25.4 -> 28.9 mm
- net LIGHT_SENSOR: track 26.1 -> 22.5 mm
- net 12V: track 10.6 -> 7.15 mm
- net Net-(R11-Pad1): track 125.3 -> 122.1 mm
- net Net-(R5-Pad2): track 124.0 -> 121.5 mm
- net GND: track 29.3 -> 30.1 mm, vias 0 -> 6
- added copper zone on B.Cu, net (none)
- added copper zone on B.Cu, net GND
- added copper zone on F.Cu, net GND
